File: pcb/pip/pip.kicad_sch (KiCad schematic)
At the start: 30 parts, among them J1 USBPCB, Q1 BC847, SW1 FLASH, SW2 RESET, SW3 BUTTON_A, SW4 BUTTON_B, U1 74HC595, U2 W25Q32JVSS, U3 CH552G

Commit message: pcb design
Parts:
- DS1: footprint Connector_PinSocket_2.54mm:PinSocket_2x05_P2.54mm_Vertical -> libraries:Display_2531AB
- J1: footprint SparkFun-Connectors:USB-A-PCB -> libraries:USB-A-PCB
- SW1, SW2: footprint Button_Switch_SMD:SW_Push_1P1T_NO_6x6mm_H9.5mm -> libraries:SW_Push_45x45mm_H1.5mm
- SW3, SW4: footprint Button_Switch_SMD:SW_Push_1P1T_NO_6x6mm_H9.5mm -> libraries:SW_TL3330AF130QG
Connections:
- net P3.6: now also J1.USB_DP (D+); no longer J1.USB_ (D-)
- net P3.7: now also J1.USB_DC (D-); no longer J1.USB_ (D-)
Changed lines of the file:
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@@
     (property "Reference" "SW1" (id 0) (at 116.84 121.92 0))
     (property "Value" "FLASH" (id 1) (at 116.84 124.46 0))
-    (property "Footprint" "Button_Switch_SMD:SW_Push_1P1T_NO_6x6mm_H9.5mm" (id 2) (at 116.84 124.46 0)
+    (property "Footprint" "libraries:SW_Push_45x45mm_H1.5mm" (id 2) (at 116.84 124.46 0)
       (effects (font (size 1.27 1.27)) hide)
     )
@@
     (pin "1")
   )
-  (symbol (lib_id "Switch:SW_MEC_5G") (at 247.65 57.15 0) (unit 1)
+  (symbol (lib_name "SW_MEC_5G_2") (lib_id "Switch:SW_MEC_5G") (at 247.65 57.15 0) (unit 1)
     (in_bom yes) (on_board yes) (fields_autoplaced)
     (property "Reference" "SW4" (id 0) (at 247.65 49.53 0))
     (property "Value" "BUTTON_B" (id 1) (at 247.65 52.07 0))
-    (property "Footprint" "Button_Switch_SMD:SW_Push_1P1T_NO_6x6mm_H9.5mm" (id 2) (at 247.65 52.07 0)
+    (property "Footprint" "libraries:SW_TL3330AF130QG" (id 2) (at 247.65 52.07 0)
       (effects (font (size 1.27 1.27)) hide)
     )
@@
       (effects (font (size 1.27 1.27)) (justify left))
     )
-    (property "Footprint" "SparkFun-Connectors:USB-A-PCB" (id 2) (at 40.132 119.38 0)
+    (property "Footprint" "libraries:USB-A-PCB" (id 2) (at 40.132 119.38 0)
       (effects (font (size 0.508 0.508)) hide)
     )
@@
     (pin "5V")
     (pin "GND")
-    (pin "USB_")
-    (pin "USB_")
+    (pin "USB_DC")
+    (pin "USB_DP")
   )
   (symbol (lib_id "power:GND") (at 34.29 125.73 0) (unit 1)
@@
     (property "Reference" "SW2" (id 0) (at 116.84 158.75 0))
     (property "Value" "RESET" (id 1) (at 116.84 161.29 0))
-    (property "Footprint" "Button_Switch_SMD:SW_Push_1P1T_NO_6x6mm_H9.5mm" (id 2) (at 116.84 161.29 0)
+    (property "Footprint" "libraries:SW_Push_45x45mm_H1.5mm" (id 2) (at 116.84 161.29 0)
       (effects (font (size 1.27 1.27)) hide)
     )
@@
     (pin "1")
   )
-  (symbol (lib_id "Switch:SW_MEC_5G") (at 247.65 43.18 0) (unit 1)
+  (symbol (lib_name "SW_MEC_5G_1") (lib_id "Switch:SW_MEC_5G") (at 247.65 43.18 0) (unit 1)
     (in_bom yes) (on_board yes) (fields_autoplaced)
     (property "Reference" "SW3" (id 0) (at 247.65 35.56 0))
     (property "Value" "BUTTON_A" (id 1) (at 247.65 38.1 0))
-    (property "Footprint" "Button_Switch_SMD:SW_Push_1P1T_NO_6x6mm_H9.5mm" (id 2) (at 247.65 38.1 0)
+    (property "Footprint" "libraries:SW_TL3330AF130QG" (id 2) (at 247.65 38.1 0)
       (effects (font (size 1.27 1.27)) hide)
     )
@@
     (property "Reference" "DS1" (id 0) (at 87.63 31.75 0))
     (property "Value" "NET-2531AB-11" (id 1) (at 87.63 34.29 0))
-    (property "Footprint" "Connector_PinSocket_2.54mm:PinSocket_2x05_P2.54mm_Vertical" (id 2) (at 87.376 66.802 0)
+    (property "Footprint" "libraries:Display_2531AB" (id 2) (at 87.376 66.802 0)
       (effects (font (size 1.27 1.27)) hide)
     )
@@
     )
     (path "/faf12075-f790-48f7-b98d-8cdc7ff36399"
-      (reference "DS1") (unit 1) (value "NET-2531AB-11") (footprint "Connector_PinSocket_2.54mm:PinSocket_2x05_P2.54mm_Vertical")
+      (reference "DS1") (unit 1) (value "NET-2531AB-11") (footprint "libraries:Display_2531AB")
     )
     (path "/a097d749-6ef8-4b1b-a562-8acb99d5e009"
-      (reference "J1") (unit 1) (value "USBPCB") (footprint "SparkFun-Connectors:USB-A-PCB")
+      (reference "J1") (unit 1) (value "USBPCB") (footprint "libraries:USB-A-PCB")
     )
     (path "/94c774b1-76b8-475d-a5dd-c801f9fcf7cc"
@@
     )
     (path "/7d57d020-6761-454a-adde-96130f7a7af0"
-      (reference "SW1") (unit 1) (value "FLASH") (footprint "Button_Switch_SMD:SW_Push_1P1T_NO_6x6mm_H9.5mm")
+      (reference "SW1") (unit 1) (value "FLASH") (footprint "libraries:SW_Push_45x45mm_H1.5mm")
     )
     (path "/b9ea31b2-7a6c-4b06-9111-2a7c49c30b95"
-      (reference "SW2") (unit 1) (value "RESET") (footprint "Button_Switch_SMD:SW_Push_1P1T_NO_6x6mm_H9.5mm")
+      (reference "SW2") (unit 1) (value "RESET") (footprint "libraries:SW_Push_45x45mm_H1.5mm")
     )
     (path "/d7636a9f-60cf-4cd0-8591-a070e8fb13de"
-      (reference "SW3") (unit 1) (value "BUTTON_A") (footprint "Button_Switch_SMD:SW_Push_1P1T_NO_6x6mm_H9.5mm")
+      (reference "SW3") (unit 1) (value "BUTTON_A") (footprint "libraries:SW_TL3330AF130QG")
     )
     (path "/82841d81-957b-4446-a71a-2cf37c28cf92"
-      (reference "SW4") (unit 1) (value "BUTTON_B") (footprint "Button_Switch_SMD:SW_Push_1P1T_NO_6x6mm_H9.5mm")
+      (reference "SW4") (unit 1) (value "BUTTON_B") (footprint "libraries:SW_TL3330AF130QG")
     )
     (path "/3f0ac564-9062-441b-a914-4153b3b592eb"
